Commit message: Fix xacro imcompatibilities

File: iiwa_description/urdf/iiwa.transmission.xacro (robot description, xacro)
@@ -24,78 +24,64 @@
   <xacro:macro name="iiwa_transmission" params="hardware_interface">
     <transmission name="${robot_name}_tran_1">
-      <robotNamespace>/${robot_name}</robotNamespace>
       <type>transmission_interface/SimpleTransmission</type>
       <joint name="${robot_name}_joint_1">
-	<hardwareInterface>hardware_interface/${hardware_interface}</hardwareInterface>
+            <hardwareInterface>hardware_interface/${hardware_interface}</hardwareInterface>
       </joint>
       <actuator name="${robot_name}_motor_1">
-	<hardwareInterface>hardware_interface/${hardware_interface}</hardwareInterface>
-	<mechanicalReduction>1</mechanicalReduction>
+            <mechanicalReduction>1</mechanicalReduction>
       </actuator>
     </transmission>
     <transmission name="${robot_name}_tran_2">
-      <robotNamespace>/${robot_name}</robotNamespace>
       <type>transmission_interface/SimpleTransmission</type>
       <joint name="${robot_name}_joint_2">
-	<hardwareInterface>hardware_interface/${hardware_interface}</hardwareInterface>
+            <hardwareInterface>hardware_interface/${hardware_interface}</hardwareInterface>
       </joint>
       <actuator name="${robot_name}_motor_2">
-	<hardwareInterface>hardware_interface/${hardware_interface}</hardwareInterface>
-	<mechanicalReduction>1</mechanicalReduction>
+            <mechanicalReduction>1</mechanicalReduction>
       </actuator>
     </transmission>
     <transmission name="${robot_name}_tran_3">
-      <robotNamespace>/${robot_name}</robotNamespace>
       <type>transmission_interface/SimpleTransmission</type>
       <joint name="${robot_name}_joint_3">
-	<hardwareInterface>hardware_interface/${hardware_interface}</hardwareInterface>
+            <hardwareInterface>hardware_interface/${hardware_interface}</hardwareInterface>
       </joint>
       <actuator name="${robot_name}_motor_3">
-	<hardwareInterface>hardware_interface/${hardware_interface}</hardwareInterface>
-	<mechanicalReduction>1</mechanicalReduction>
+            <mechanicalReduction>1</mechanicalReduction>
       </actuator>
     </transmission>
     <transmission name="${robot_name}_tran_4">
-      <robotNamespace>/${robot_name}</robotNamespace>
       <type>transmission_interface/SimpleTransmission</type>
       <joint name="${robot_name}_joint_4">
-	<hardwareInterface>hardware_interface/${hardware_interface}</hardwareInterface>
+            <hardwareInterface>hardware_interface/${hardware_interface}</hardwareInterface>
       </joint>
       <actuator name="${robot_name}_motor_4">
-	<hardwareInterface>hardware_interface/${hardware_interface}</hardwareInterface>
-	<mechanicalReduction>1</mechanicalReduction>
+            <mechanicalReduction>1</mechanicalReduction>
       </actuator>
     </transmission>
     <transmission name="${robot_name}_tran_5">
-      <robotNamespace>/${robot_name}</robotNamespace>
       <type>transmission_interface/SimpleTransmission</type>
       <joint name="${robot_name}_joint_5">
-	<hardwareInterface>hardware_interface/${hardware_interface}</hardwareInterface>
+            <hardwareInterface>hardware_interface/${hardware_interface}</hardwareInterface>
       </joint>
       <actuator name="${robot_name}_motor_5">
-	<hardwareInterface>hardware_interface/${hardware_interface}</hardwareInterface>
-	<mechanicalReduction>1</mechanicalReduction>
+            <mechanicalReduction>1</mechanicalReduction>
       </actuator>
     </transmission>
     <transmission name="${robot_name}_tran_6">
-      <robotNamespace>/${robot_name}</robotNamespace>
       <type>transmission_interface/SimpleTransmission</type>
       <joint name="${robot_name}_joint_6">
-	<hardwareInterface>hardware_interface/${hardware_interface}</hardwareInterface>
+            <hardwareInterface>hardware_interface/${hardware_interface}</hardwareInterface>
       </joint>
       <actuator name="${robot_name}_motor_6">
-	<hardwareInterface>hardware_interface/${hardware_interface}</hardwareInterface>
-	<mechanicalReduction>1</mechanicalReduction>
+            <mechanicalReduction>1</mechanicalReduction>
       </actuator>
     </transmission>
     <transmission name="${robot_name}_tran_7">
-      <robotNamespace>/${robot_name}</robotNamespace>
       <type>transmission_interface/SimpleTransmission</type>
       <joint name="${robot_name}_joint_7">
-	<hardwareInterface>hardware_interface/${hardware_interface}</hardwareInterface>
+            <hardwareInterface>hardware_interface/${hardware_interface}</hardwareInterface>
       </joint>
       <actuator name="${robot_name}_motor_7">
-	<hardwareInterface>hardware_interface/${hardware_interface}</hardwareInterface>
-	<mechanicalReduction>1</mechanicalReduction>
+            <mechanicalReduction>1</mechanicalReduction>
       </actuator>
     </transmission>

File: iiwa_description/urdf/iiwa14.xacro (robot description, xacro)
@@ -62,5 +62,5 @@
     <!--joint between {parent} and link_0-->
     <joint name="${parent}_${robot_name}_joint" type="fixed">
-      <xacro:insert_block name="origin"/>
+      <!-- <xacro:insert_block name="origin"/> -->
       <parent link="${parent}"/>
       <child link="${robot_name}_link_0"/>
@@ -84,12 +84,5 @@
           <mesh filename="package://iiwa_description/meshes/iiwa14/collision/link_0${collision_postfix}.stl"/>
         </geometry>
-        <material name="Grey"/>
-      </collision>
-      <self_collision_checking>
-        <origin xyz="0 0 0" rpy="0 0 0"/>
-        <geometry>
-          <capsule radius="0.15" length="0.25"/>
-        </geometry>
-      </self_collision_checking>
+      </collision>
     </link>
     <!-- joint between link_0 and link_1 -->
@@ -126,5 +119,4 @@
           <mesh filename="package://iiwa_description/meshes/iiwa14/collision/link_1${collision_postfix}.stl"/>
         </geometry>
-        <material name="Orange"/>
       </collision>
     </link>
@@ -162,5 +154,4 @@
           <mesh filename="package://iiwa_description/meshes/iiwa14/collision/link_2${collision_postfix}.stl"/>
         </geometry>
-        <material name="Orange"/>
       </collision>
     </link>
@@ -198,5 +189,4 @@
           <mesh filename="package://iiwa_description/meshes/iiwa14/collision/link_3${collision_postfix}.stl"/>
         </geometry>
-        <material name="Orange"/>
       </collision>
     </link>
@@ -234,5 +224,4 @@
           <mesh filename="package://iiwa_description/meshes/iiwa14/collision/link_4${collision_postfix}.stl"/>
         </geometry>
-        <material name="Orange"/>
       </collision>
     </link>
@@ -270,5 +259,4 @@
           <mesh filename="package://iiwa_description/meshes/iiwa14/collision/link_5${collision_postfix}.stl"/>
         </geometry>
-        <material name="Orange"/>
       </collision>
     </link>
@@ -306,5 +294,4 @@
           <mesh filename="package://iiwa_description/meshes/iiwa14/collision/link_6${collision_postfix}.stl"/>
         </geometry>
-        <material name="Orange"/>
       </collision>
     </link>
@@ -342,5 +329,4 @@
           <mesh filename="package://iiwa_description/meshes/iiwa14/collision/link_7${collision_postfix}.stl"/>
         </geometry>
-        <material name="Grey"/>
       </collision>
     </link>
